File: esp_coaster.sch (EAGLE design)
At the start: 21 parts, among them IC1 ESP-12E/F, U1 MC34063AP

Commit message: Revert "add mc34063AP"
This reverts commit ce2e4ae2c6462f3cc229f7f57adec7c62f3c656d.
Parts:
- removed C3, C4, C5: (no value), resistor:CPOL-US085CS-1AR
- removed D1: 1N5819-B, diode:1N5819-B
- removed L1: (no value), resistor:L-US0204/5
- removed R6, R7, R8: (no value), rcl:R-US_M2309
- removed U1: MC34063AP, MC34063AP:MC34063AP
Connections:
- removed net N$10: D1.A, L1.2, U1.SW_C
- removed net N$11: R6.2, R7.2, U1.COMPARATOR_NEG
- removed net N$8: C5.+, U1.CT
- removed net N$9: L1.1, R8.1, U1.DRVR_C, U1.IPK
- removed net VIN: C4.+, R8.2, U1.VCC
- removed net VOUT: C3.-, D1.C, R6.1
- net GND: no longer C3.+, C4.-, C5.-, R7.1, U1.GND, U1.SW_E
Other:
- moved on the sheet: AMS1117(3.3V), C1, C2, IC1, R1, R2, R3, R4, R5, S1, S2
