File: ESP12E_Smart_Coaster.kicad_sch (KiCad schematic)
At the start: 49 parts, among them J1 SPI_Header, J2 MLX90614 Temp Sensor, J3 Programming_header, J4 Power_Input_Header, Q1 SI2302, SW1 SW_SPDT, SW2 SW_Push, U1 T6845C_Module, U2 AMS1117-3.3, U3 ESP-12E

Commit message: Added graphics
Parts:
- added C15: 100uF, Capacitor_SMD:C_1206_3216Metric_Pad1.33x1.80mm_HandSolder, symbol Device:C_Small
Connections:
- net +5V: now also C15.1
- net GND: now also C15.2
Changed lines of the file:
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@@
   (junction (at 247.396 152.908) (diameter 0) (color 0 0 0 0)
+  )
+  (junction (at 33.782 145.288) (diameter 0) (color 0 0 0 0)
   )
   (junction (at 228.346 132.588) (diameter 0) (color 0 0 0 0)
@@
     (stroke (width 0) (type default) (color 0 0 0 0))
   )
-  (wire (pts (xy 36.576 145.288) (xy 31.496 145.288))
+  (wire (pts (xy 36.576 145.288) (xy 33.782 145.288))
+    (stroke (width 0) (type default) (color 0 0 0 0))
+  )
+  (wire (pts (xy 33.782 145.288) (xy 31.496 145.288))
     (stroke (width 0) (type default) (color 0 0 0 0))
   )
@@
     (stroke (width 0) (type default) (color 0 0 0 0))
   )
+  (wire (pts (xy 33.782 152.146) (xy 33.782 151.638))
+    (stroke (width 0) (type default) (color 0 0 0 0))
+  )
   (wire (pts (xy 196.342 75.946) (xy 200.152 75.946))
     (stroke (width 0) (type default) (color 0 0 0 0))
@@
   )
   (wire (pts (xy 228.346 126.238) (xy 228.346 132.588))
+    (stroke (width 0) (type default) (color 0 0 0 0))
+  )
+  (wire (pts (xy 33.782 146.558) (xy 33.782 145.288))
     (stroke (width 0) (type default) (color 0 0 0 0))
   )
@@
     (pin "2")
   )
+  (symbol (lib_id "Device:C_Small") (at 33.782 149.098 0) (unit 1)
+    (in_bom yes) (on_board yes)
+    (property "Reference" "C15" (id 0) (at 28.956 150.876 0)
+      (effects (font (size 1 1)) (justify left))
+    )
+    (property "Value" "100uF" (id 1) (at 27.432 148.844 0)
+      (effects (font (size 1 1)) (justify left))
+    )
+    (property "Footprint" "Capacitor_SMD:C_1206_3216Metric_Pad1.33x1.80mm_HandSolder" (id 2) (at 33.782 149.098 0)
+      (effects (font (size 1.27 1.27)) hide)
+    )
+    (property "Datasheet" "~" (id 3) (at 33.782 149.098 0)
+      (effects (font (size 1.27 1.27)) hide)
+    )
+    (pin "1")
+    (pin "2")
+  )
   (symbol (lib_id "Device:C_Small") (at 114.046 132.588 270) (unit 1)
     (in_bom yes) (on_board yes)
@@
     (pin "1")
     (pin "2")
+  )
+  (symbol (lib_id "power:GND") (at 33.782 152.146 0) (unit 1)
+    (in_bom yes) (on_board yes)
+    (property "Reference" "#PWR035" (id 0) (at 33.782 158.496 0)
+      (effects (font (size 1.27 1.27)) hide)
+    )
+    (property "Value" "GND" (id 1) (at 33.782 155.956 0))
+    (property "Footprint" "" (id 2) (at 33.782 152.146 0)
+      (effects (font (size 1.27 1.27)) hide)
+    )
+    (property "Datasheet" "" (id 3) (at 33.782 152.146 0)
+      (effects (font (size 1.27 1.27)) hide)
+    )
+    (pin "1")
   )
   (symbol (lib_id "Device:C_Small") (at 149.606 132.588 270) (unit 1)
@@
       (reference "#PWR034") (unit 1) (value "GND") (footprint "")
     )
+    (path "/c66e44f7-c7f5-479d-95a7-eff71fcb2267"
+      (reference "#PWR035") (unit 1) (value "GND") (footprint "")
+    )
     (path "/d726cd84-e307-4fc7-9889-3524b9a9ac3d"
       (reference "BT1") (unit 1) (value "Battery") (footprint "Battery:BatteryHolder_Keystone_1042_1x18650")
@@
       (reference "C14") (unit 1) (value "0.1uF") (footprint "Capacitor_SMD:C_1206_3216Metric_Pad1.33x1.80mm_HandSolder")
     )
+    (path "/b14311f1-8112-4eb9-9a61-b0029ab2f58f"
+      (reference "C15") (unit 1) (value "100uF") (footprint "Capacitor_SMD:C_1206_3216Metric_Pad1.33x1.80mm_HandSolder")
+    )
     (path "/3c754d4d-830e-4be9-96d7-fdda182a0183"
